File: T_pcb_ca_ca/ca_ca.brd (EAGLE design)
At the start: 100 x 80 mm, 14 parts, among them IC1 74AS04N, IC2 74ALS02N, T1 BT138-V

Commit message: Add files via upload
Parts:
- removed C1: (no value), rcl:C102-064X133
- removed IC1: 74AS04N, 74xx-us:DIL14
- removed JP1: (no value), pinhead:1X02
- removed JP2: (no value), pinhead:1X05
- removed T1: BT138-V, triac:TO220BV
- added C4, C5, CC1, CC2: (no value), rcl:C102-064X133
- added CONECT1: (no value), pinhead:1X02
- added D1, D2: 1N4004, diode:DO41-10
- added IC3, IC4: 74AS04N, 74xx-us:DIL14
- added JP3: (no value), pinhead:1X05
- added OK3: MOC3020M, optocoupler:DIL06
- added RR1, RR2, RR3, RR4: (no value), rcl:0617/22
- added T2: BT138-V, triac:TO220BV
- added TP1, TP2: TPPAD1-17Y, testpad:P1-17Y
- OK1: value MOC3010M -> 4N33
- R4: device rcl:0204/5 -> rcl:0617/22
- moved X2 116.5 mm to (72.4, 62.2), turned to 270 degrees
- moved X1 112.8 mm to (72.4, 73.7), turned to 270 degrees
- moved R4 92.5 mm to (48.3, 31.8), turned to 90 degrees
- moved IC2 86.5 mm to (63.5, 26.7)
- moved OK1 78.2 mm to (31.8, 24.1)
- moved R2 68.4 mm to (40.6, 31.8), turned to 270 degrees
- moved OK2 52.6 mm to (31.8, 38.1)
- moved R3 48.6 mm to (15.2, 31.8), turned to 90 degrees
- moved R1 35.4 mm to (8.89, 31.8), turned to 90 degrees
Connections:
- new net N$1: OK3.1, RR1.2
- new net N$10: IC2.2, IC3.2, JP3.3
- new net N$11: IC4.1, OK2.5, R4.2
- new net N$12: D2.C, OK2.1, R3.2
- new net N$13: IC2.3, IC4.2, JP3.4
- new net N$14: IC2.1, JP3.2
- new net N$2: CONECT1.2, RR1.1
- new net N$3: OK3.4, T2.G
- new net N$4: CC1.1, RR2.1, RR3.2
- new net N$5: OK3.6, RR2.2
- new net N$6: IC3.1, OK1.5, R2.2
- new net N$7: CC1.2, CC2.2, T2.T1, X2.2
- new net N$8: CC2.1, RR4.2
- new net N$9: D1.C, OK1.1, R1.2
- new net V+: D2.A, OK2.2, R1.1, RR3.1, RR4.1, T2.T2, TP1.TP, X1.1
- new net V-: D1.A, OK1.2, R3.1, TP2.TP, X1.2, X2.1
- new net VDD: C4.1, C5.1, IC3.14, IC4.14, JP3.1, R2.1, R4.1
- net GND: now also C4.2, C5.2, CONECT1.1, IC3.7, IC4.7, JP3.5, OK1.4, OK2.4, OK3.2; no longer IC1.7
- net VCC: no longer IC1.14
Routing:
- net V+: track 0.00 -> 209.3 mm
- net GND: track 0.00 -> 190.2 mm
- net V-: track 0.00 -> 186.6 mm
- net N$7: track 0.00 -> 100.7 mm
- net VDD: track 0.00 -> 87.6 mm
- net N$11: track 0.00 -> 81.9 mm
- net N$13: track 0.00 -> 71.1 mm
- net N$6: track 0.00 -> 60.3 mm
- net N$4: track 0.00 -> 47.6 mm
- net N$9: track 0.00 -> 45.1 mm
- net N$10: track 0.00 -> 42.5 mm
- net N$12: track 0.00 -> 36.5 mm
- net N$8: track 0.00 -> 32.7 mm
- net N$1: track 0.00 -> 29.9 mm
- net N$14: track 0.00 -> 25.9 mm
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Other:
- board size 100 x 80 mm -> 79.7 x 71.1 mm
