File: T_pcb_ca_ca/ca_ca.sch (EAGLE design)
At the start: 14 parts, among them IC1 74AS04N, IC2 74ALS02N, T1 BT138-V

Commit message: Add files via upload
Parts:
- removed C1: (no value), rcl:C-US102-064X133
- removed IC1: 74AS04N, 74xx-us:74AS04N
- removed JP1: (no value), pinhead:PINHD-1X2
- removed JP2: (no value), pinhead:PINHD-1X5
- removed R3: (no value), rcl:R-US_0617/22
- removed R4: (no value), rcl:R-US_0204/5
- removed T1: BT138-V, triac:BT138-V
- added C4, C5, CC1, CC2: (no value), rcl:C-US102-064X133
- added CONECT1: (no value), pinhead:PINHD-1X2
- added D1, D2: 1N4004, diode:1N4004
- added IC3, IC4: 74AS04N, 74xx-us:74AS04N
- added JP3: (no value), pinhead:PINHD-1X5
- added OK3: MOC3020M, optocoupler:MOC3020M
- added R8, R9, RR1, RR2, RR3, RR4: (no value), rcl:R-US_0617/22
- added T2: BT138-V, triac:BT138-V
- OK1: value MOC3010M -> 4N33; device optocoupler:MOC3010M -> optocoupler:4N33
Connections:
- new net GND: C4.2, C5.2, CONECT1.1, IC3P.GND, IC4P.GND, JP3.5, OK1.E, OK2.E, OK3.C
- new net N$1: OK3.A, RR1.2
- new net N$10: IC2A.I0, IC3A.O, JP3.3
- new net N$11: IC4A.I, OK1.COL, R9.2
- new net N$12: D2.C, OK1.A, R8.2
- new net N$13: IC2A.I1, IC4A.O, JP3.4
- new net N$14: IC2A.O, JP3.2
- new net N$2: CONECT1.2, RR1.1
- new net N$3: OK3.A1, T2.G
- new net N$4: CC1.1, RR2.1, RR3.2
- new net N$5: OK3.A2, RR2.2
- new net N$6: IC3A.I, OK2.COL, R2.2
- new net N$7: CC1.2, CC2.2, T2.A1, X2-2.KL
- new net N$8: CC2.1, RR4.2
- new net N$9: D1.C, OK2.A, R1.2
- new net V+: D2.A, OK1.C, R1.1, RR3.1, RR4.1, T2.A2, X1-1.KL
- new net V-: D1.A, OK2.C, R8.1, X1-2.KL, X2-1.KL
- new net VDD: C4.1, C5.1, IC3P.VCC, IC4P.VCC, JP3.1, R2.1, R9.1
Other:
- moved on the sheet: IC2A, OK2, R1, R2, X1-1, X1-2, X2-1, X2-2

Commit message: Add files via upload
Parts:
- added TP1, TP2: TPPAD1-17Y, testpad:TPPAD1-17Y
- renumbered R8 to R3, R9 to R4
Connections:
- net N$11: now also OK2.COL; no longer OK1.COL
- net N$12: now also OK2.A; no longer OK1.A
- net N$6: now also OK1.COL; no longer OK2.COL
- net N$9: now also OK1.A; no longer OK2.A
- net V+: now also OK2.C, TP1.TP; no longer OK1.C
- net V-: now also OK1.C, TP2.TP; no longer OK2.C
Other:
- moved on the sheet: OK1, OK2
Changed lines of the file:
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@@
 <part name="R2" library="rcl" library_urn="urn:adsk.eagle:library:334" deviceset="R-US_" device="0617/22" package3d_urn="urn:adsk.eagle:package:23577/1"/>
 <part name="CONECT1" library="pinhead" library_urn="urn:adsk.eagle:library:325" deviceset="PINHD-1X2" device="" package3d_urn="urn:adsk.eagle:package:22435/2"/>
-<part name="OK2" library="optocoupler" library_urn="urn:adsk.eagle:library:320" deviceset="4N33" device="" package3d_urn="urn:adsk.eagle:package:21942/1"/>
+<part name="OK1" library="optocoupler" library_urn="urn:adsk.eagle:library:320" deviceset="4N33" device="" package3d_urn="urn:adsk.eagle:package:21942/1"/>
 <part name="SUPPLY1" library="supply2" library_urn="urn:adsk.eagle:library:372" deviceset="VDD" device=""/>
 <part name="GND1" library="supply1" library_urn="urn:adsk.eagle:library:371" deviceset="GND" device=""/>
@@
 <part name="IC4" library="74xx-us" library_urn="urn:adsk.eagle:library:88" deviceset="74*04" device="N" package3d_urn="urn:adsk.eagle:package:16407/2" technology="AS"/>
 <part name="GND3" library="supply1" library_urn="urn:adsk.eagle:library:371" deviceset="GND" device=""/>
-<part name="R8" library="rcl" library_urn="urn:adsk.eagle:library:334" deviceset="R-US_" device="0617/22" package3d_urn="urn:adsk.eagle:package:23577/1"/>
-<part name="R9" library="rcl" library_urn="urn:adsk.eagle:library:334" deviceset="R-US_" device="0617/22" package3d_urn="urn:adsk.eagle:package:23577/1"/>
-<part name="OK1" library="optocoupler" library_urn="urn:adsk.eagle:library:320" deviceset="4N33" device="" package3d_urn="urn:adsk.eagle:package:21942/1"/>
+<part name="R3" library="rcl" library_urn="urn:adsk.eagle:library:334" deviceset="R-US_" device="0617/22" package3d_urn="urn:adsk.eagle:package:23577/1"/>
+<part name="R4" library="rcl" library_urn="urn:adsk.eagle:library:334" deviceset="R-US_" device="0617/22" package3d_urn="urn:adsk.eagle:package:23577/1"/>
+<part name="OK2" library="optocoupler" library_urn="urn:adsk.eagle:library:320" deviceset="4N33" device="" package3d_urn="urn:adsk.eagle:package:21942/1"/>
 <part name="SUPPLY2" library="supply2" library_urn="urn:adsk.eagle:library:372" deviceset="VDD" device=""/>
 <part name="P+3" library="supply1" library_urn="urn:adsk.eagle:library:371" deviceset="V+" device=""/>
@@
 <part name="RR2" library="rcl" library_urn="urn:adsk.eagle:library:334" deviceset="R-US_" device="0617/22" package3d_urn="urn:adsk.eagle:package:23577/1"/>
 <part name="RR4" library="rcl" library_urn="urn:adsk.eagle:library:334" deviceset="R-US_" device="0617/22" package3d_urn="urn:adsk.eagle:package:23577/1"/>
+<part name="TP1" library="testpad" library_urn="urn:adsk.eagle:library:385" deviceset="TP" device="PAD1-17Y" package3d_urn="urn:adsk.eagle:package:27953/1"/>
+<part name="TP2" library="testpad" library_urn="urn:adsk.eagle:library:385" deviceset="TP" device="PAD1-17Y" package3d_urn="urn:adsk.eagle:package:27953/1"/>
 </parts>
 <sheets>
@@
 <attribute name="VALUE" x="-57.15" y="121.92" size="1.778" layer="96" rot="R180"/>
 </instance>
-<instance part="OK2" gate="A" x="-22.86" y="53.34" smashed="yes">
+<instance part="OK1" gate="A" x="-22.86" y="53.34" smashed="yes">
 <attribute name="NAME" x="-29.8704" y="61.5696" size="1.778" layer="95"/>
 <attribute name="VALUE" x="-29.8704" y="45.7962" size="1.778" layer="96"/>
@@
 <attribute name="VALUE" x="-12.7" y="43.18" size="1.778" layer="96"/>
 </instance>
-<instance part="R8" gate="G$1" x="-60.96" y="17.78" smashed="yes">
+<instance part="R3" gate="G$1" x="-60.96" y="17.78" smashed="yes">
 <attribute name="NAME" x="-64.77" y="19.2786" size="1.778" layer="95"/>
 <attribute name="VALUE" x="-64.77" y="14.478" size="1.778" layer="96"/>
 </instance>
-<instance part="R9" gate="G$1" x="-2.54" y="22.86" smashed="yes" rot="R270">
+<instance part="R4" gate="G$1" x="-2.54" y="22.86" smashed="yes" rot="R270">
 <attribute name="NAME" x="-1.0414" y="26.67" size="1.778" layer="95" rot="R270"/>
 <attribute name="VALUE" x="-5.842" y="26.67" size="1.778" layer="96" rot="R270"/>
 </instance>
-<instance part="OK1" gate="A" x="-22.86" y="12.7" smashed="yes">
+<instance part="OK2" gate="A" x="-22.86" y="12.7" smashed="yes">
 <attribute name="NAME" x="-29.8704" y="20.9296" size="1.778" layer="95"/>
 <attribute name="VALUE" x="-29.8704" y="5.1562" size="1.778" layer="96"/>
@@
 <attribute name="NAME" x="47.2186" y="120.65" size="1.778" layer="95" rot="R270"/>
 <attribute name="VALUE" x="42.418" y="120.65" size="1.778" layer="96" rot="R270"/>
+</instance>
+<instance part="TP1" gate="G$1" x="-71.12" y="63.5" smashed="yes">
+<attribute name="NAME" x="-72.39" y="64.77" size="1.778" layer="95"/>
+<attribute name="TP_SIGNAL_NAME" x="-69.85" y="62.23" size="1.778" layer="97"/>
+</instance>
+<instance part="TP2" gate="G$1" x="-71.12" y="50.8" smashed="yes">
+<attribute name="NAME" x="-72.39" y="52.07" size="1.778" layer="95"/>
+<attribute name="TP_SIGNAL_NAME" x="-69.85" y="49.53" size="1.778" layer="97"/>
 </instance>
 </instances>
@@
 <segment>
 <pinref part="GND3" gate="1" pin="GND"/>
-<pinref part="OK2" gate="A" pin="E"/>
+<pinref part="OK1" gate="A" pin="E"/>
 <wire x1="-10.16" y1="48.26" x2="-10.16" y2="50.8" width="0.1524" layer="91"/>
 <wire x1="-10.16" y1="50.8" x2="-15.24" y2="50.8" width="0.1524" layer="91"/>
@@
 <segment>
 <pinref part="GND4" gate="1" pin="GND"/>
-<pinref part="OK1" gate="A" pin="E"/>
+<pinref part="OK2" gate="A" pin="E"/>
 <wire x1="-10.16" y1="7.62" x2="-10.16" y2="10.16" width="0.1524" layer="91"/>
 <wire x1="-10.16" y1="10.16" x2="-15.24" y2="10.16" width="0.1524" layer="91"/>
@@
 <pinref part="P+2" gate="1" pin="V+"/>
 <pinref part="R1" gate="G$1" pin="1"/>
-<wire x1="-76.2" y1="58.42" x2="-66.04" y2="58.42" width="0.1524" layer="91"/>
-</segment>
-<segment>
-<pinref part="OK1" gate="A" pin="C"/>
+<wire x1="-76.2" y1="58.42" x2="-71.12" y2="58.42" width="0.1524" layer="91"/>
+<pinref part="TP1" gate="G$1" pin="TP"/>
+<wire x1="-71.12" y1="58.42" x2="-66.04" y2="58.42" width="0.1524" layer="91"/>
+<wire x1="-71.12" y1="60.96" x2="-71.12" y2="58.42" width="0.1524" layer="91"/>
+<junction x="-71.12" y="58.42"/>
+</segment>
+<segment>
+<pinref part="OK2" gate="A" pin="C"/>
 <pinref part="D2" gate="1" pin="A"/>
 <wire x1="-33.02" y1="10.16" x2="-45.72" y2="10.16" width="0.1524" layer="91"/>
@@
 </segment>
 <segment>
-<pinref part="OK2" gate="A" pin="C"/>
+<pinref part="OK1" gate="A" pin="C"/>
 <pinref part="D1" gate="1" pin="A"/>
 <wire x1="-33.02" y1="50.8" x2="-45.72" y2="50.8" width="0.1524" layer="91"/>
 <wire x1="-45.72" y1="50.8" x2="-45.72" y2="45.72" width="0.1524" layer="91"/>
 <pinref part="P-2" gate="1" pin="V-"/>
-<wire x1="-45.72" y1="45.72" x2="-76.2" y2="45.72" width="0.1524" layer="91"/>
+<wire x1="-45.72" y1="45.72" x2="-71.12" y2="45.72" width="0.1524" layer="91"/>
 <junction x="-45.72" y="50.8"/>
+<pinref part="TP2" gate="G$1" pin="TP"/>
+<wire x1="-71.12" y1="45.72" x2="-76.2" y2="45.72" width="0.1524" layer="91"/>
+<wire x1="-71.12" y1="48.26" x2="-71.12" y2="45.72" width="0.1524" layer="91"/>
+<junction x="-71.12" y="45.72"/>
 </segment>
 <segment>
 <pinref part="P-3" gate="1" pin="V-"/>
-<pinref part="R8" gate="G$1" pin="1"/>
+<pinref part="R3" gate="G$1" pin="1"/>
 <wire x1="-73.66" y1="17.78" x2="-66.04" y2="17.78" width="0.1524" layer="91"/>
 </segment>
@@
 <segment>
 <pinref part="SUPPLY2" gate="G$1" pin="VDD"/>
-<pinref part="R9" gate="G$1" pin="1"/>
+<pinref part="R4" gate="G$1" pin="1"/>
 <wire x1="-2.54" y1="30.48" x2="-2.54" y2="27.94" width="0.1524" layer="91"/>
 </segment>
@@
 <segment>
 <pinref part="R2" gate="G$1" pin="2"/>
-<pinref part="OK2" gate="A" pin="COL"/>
+<pinref part="OK1" gate="A" pin="COL"/>
 <wire x1="-2.54" y1="58.42" x2="-2.54" y2="55.88" width="0.1524" layer="91"/>
 <wire x1="-2.54" y1="55.88" x2="-15.24" y2="55.88" width="0.1524" layer="91"/>
@@
 <pinref part="D1" gate="1" pin="C"/>
 <wire x1="-45.72" y1="58.42" x2="-45.72" y2="55.88" width="0.1524" layer="91"/>
-<pinref part="OK2" gate="A" pin="A"/>
+<pinref part="OK1" gate="A" pin="A"/>
 <wire x1="-45.72" y1="58.42" x2="-33.02" y2="58.42" width="0.1524" layer="91"/>
 <junction x="-45.72" y="58.42"/>
@@
 <net name="N$11" class="0">
 <segment>
-<pinref part="R9" gate="G$1" pin="2"/>
-<pinref part="OK1" gate="A" pin="COL"/>
+<pinref part="R4" gate="G$1" pin="2"/>
+<pinref part="OK2" gate="A" pin="COL"/>
 <wire x1="-2.54" y1="17.78" x2="-2.54" y2="15.24" width="0.1524" layer="91"/>
 <wire x1="-2.54" y1="15.24" x2="-15.24" y2="15.24" width="0.1524" layer="91"/>
@@
 <net name="N$12" class="0">
 <segment>
-<pinref part="R8" gate="G$1" pin="2"/>
+<pinref part="R3" gate="G$1" pin="2"/>
 <wire x1="-55.88" y1="17.78" x2="-45.72" y2="17.78" width="0.1524" layer="91"/>
 <pinref part="D2" gate="1" pin="C"/>
 <wire x1="-45.72" y1="17.78" x2="-45.72" y2="15.24" width="0.1524" layer="91"/>
-<pinref part="OK1" gate="A" pin="A"/>
+<pinref part="OK2" gate="A" pin="A"/>
 <wire x1="-45.72" y1="17.78" x2="-33.02" y2="17.78" width="0.1524" layer="91"/>
 <junction x="-45.72" y="17.78"/>
